File: Bina_Badge.kicad_pcb (KiCad board)
At the start: 2 copper layers, 50 x 50 mm, 20 parts, among them J1 Conn_01x06, P1 USB_C_Plug_USB2.0, SW1 SW_Push, U1 ATtiny85-20S

Commit message: production ready
Parts:
- D10: value 1N4148WS -> SM4007; footprint Diode_SMD:D_SOD-323 -> Diode_SMD:D_MELF
- moved D10 1.06 mm to (142.5, 91.0)
Other:
- board text added: "01010101 00100000 01001111 00100000 01101101 01100101"
- board text added: "01100001 00100000 01100100 01110010 01101001 01101110 01101011"
